Commit message: Add files via upload

File: ruka_description/urdf/gripper_bunka.xacro (robot description, xacro)
@@ -6,8 +6,3 @@
     <xacro:include filename="$(find ruka_description)/urdf/gripper_macro.xacro"/>
     <xacro:gripper_macro prefix=""/>
-    <joint name="dobot_gripper_joint" type="fixed">
-        <origin xyz="0 0 0" rpy="0 0 0" />
-        <parent link="Link6" />
-        <child  link="gripper" /> <!--gripper-->
-    </joint>
 </robot>

File: ruka_description/urdf/gripper_macro.xacro (robot description, xacro)
@@ -2,4 +2,9 @@
 <robot xmlns:xacro="http://www.ros.org/wiki/xacro">
     <xacro:macro name="gripper_macro" params="prefix">
+    <joint name="dobot_gripper_joint" type="fixed">
+        <origin xyz="0 0 0" rpy="0 0 0" />
+        <parent link="Link6" />
+        <child  link="gripper" /> <!--gripper-->
+    </joint>
         <link name="${prefix}gripper">
           <inertial>
@@ -36,4 +41,10 @@
           </collision>
       </link>
+    <joint name="tcp_joint" type="fixed">
+        <origin xyz="0 0.2 0.2" rpy="0 0 0" />
+        <parent link="gripper" />
+        <child  link="tcp" /> <!--gripper -->
+    </joint>
+    <link name="tcp"/>
         <!-- Add joints, inertial properties, etc. as needed -->
   </xacro:macro>
