Commit message: Add files via upload

File: ruka_description/urdf/gripper_macro.xacro (robot description, xacro)
@@ -2,9 +2,4 @@
 <robot xmlns:xacro="http://www.ros.org/wiki/xacro">
     <xacro:macro name="gripper_macro" params="prefix">
-    <joint name="dobot_gripper_joint" type="fixed">
-        <origin xyz="0 0 0" rpy="0 0 0" />
-        <parent link="Link6" />
-        <child  link="gripper" /> <!--gripper-->
-    </joint>
         <link name="${prefix}gripper">
           <inertial>
@@ -41,11 +36,19 @@
           </collision>
       </link>
-    <joint name="tcp_joint" type="fixed">
-        <origin xyz="0 0.2 0.2" rpy="0 0 0" />
-        <parent link="gripper" />
-        <child  link="tcp" /> <!--gripper -->
+    <joint name="dobot_gripper_joint" type="fixed">
+        <origin xyz="0 0 0" rpy="0 0 0"/>
+        <parent link="Link6"/>
+        <child link="gripper"/>
     </joint>
-    <link name="tcp"/>
-        <!-- Add joints, inertial properties, etc. as needed -->
+<joint name="tcp_joint" type="fixed">
+    <origin xyz="-0.105 0 0.065" rpy="0 3.1416 1.5708" />
+    <parent link="gripper" />
+    <child link="tcp" />
+</joint>
+<link name="tcp"/>
+        <!--90 degrees: rpy="0 0 1.5708"
+180 degrees: rpy="0 0 3.1416"
+270 degrees: rpy="0 0 4.7124"
+360 degrees: rpy="0 0 6.2832 Add joints, inertial properties, etc. as needed -->
   </xacro:macro>
 </robot>

Commit message: Add files via upload

File: ruka_description/urdf/gripper_macro.xacro (robot description, xacro)
@@ -21,5 +21,5 @@
                   rpy="0 0 0" />
               <geometry>
-                  <mesh scale = "0.001 0.001 0.001" filename="package://ruka_description/meshes/gripper/Gripper_1.4_mod_s_vzduch_pris.STL" />
+                  <mesh scale = "0.0001 0.0001 0.0001" filename="package://ruka_description/meshes/gripper/Gripper_1.5REALSTLORIGINALIGNv3.stl" />
               </geometry>
               <material name="">
@@ -32,10 +32,10 @@
                   rpy="0 0 0" />
               <geometry>
-                  <mesh scale = "0.001 0.001 0.001" filename="package://ruka_description/meshes/gripper/Gripper_1.4_mod_s_vzduch_pris.STL" />
+                  <mesh scale = "0.0001 0.0001 0.0001" filename="package://ruka_description/meshes/gripper/Gripper_1.5REALSTLORIGINALIGNv3.stl" />
               </geometry>
           </collision>
       </link>
     <joint name="dobot_gripper_joint" type="fixed">
-        <origin xyz="0 0 0" rpy="0 0 0"/>
+        <origin xyz="0 0 0" rpy="0 0 1.5708"/>
         <parent link="Link6"/>
         <child link="gripper"/>
