Commit message: tf

File: ruka_description/urdf/bunka.urdf (robot description, URDF)
Before this commit: robot cr5_robot, 10 links, 9 joints
Links:
- removed link dummy_link
- added link world
Joints:
- joint dummy_joint: parent dummy_link -> world
- joint tcp_joint: origin xyz=-0.105 0 0.065 rpy=0 3.1416 1.5708 -> xyz=-0.105 0 0.065 rpy=-1.5708 0 1.5708

File: ruka_description/urdf/dobot_macro.xacro (robot description, xacro)
@@ -3,5 +3,5 @@
 <!--params neviem ci tammaju byt <xacro:include filename = "cr5_robot">-->
   <xacro:macro name="cr5_robot" params="prefix">
-      <link name="${prefix}dummy_link"/>
+      <link name="world"/>
       <link name="${prefix}base_link">
           <inertial>
@@ -39,5 +39,5 @@
       </link>
       <joint name="${prefix}dummy_joint" type="fixed">
-          <parent link="${prefix}dummy_link" />
+          <parent link="world" />
           <child link="${prefix}base_link" />
       </joint>

File: ruka_description/urdf/gripper_macro.xacro (robot description, xacro)
@@ -42,5 +42,5 @@
     </joint>
 <joint name="tcp_joint" type="fixed">
-    <origin xyz="-0.105 0 0.065" rpy="0 3.1416 1.5708" />
+    <origin xyz="-0.105 0 0.065" rpy="-1.5708 0 1.5708" />
     <parent link="gripper" />
     <child link="tcp" />

File: ruka_moveit_config_real_gripper/config/gazebo_cr5_robot.urdf (robot description, URDF)
Before this commit: robot cr5_robot, 10 links, 9 joints
Links:
- removed link dummy_link
- added link world
Joints:
- joint dummy_joint: parent dummy_link -> world
